File: Cantor_Classic/backplate.kicad_pcb (KiCad board)
At the start: 2 copper layers, 138.8 x 89.9 mm, 0 parts

Commit message: [REL]v1
Parts:
- added G***: LOGO, kdkb_tools:KBKD_cantor, F.Cu at (152.0, 100.5)
- added G***: LOGO, kdkb_tools:KBKD_cantor, B.Cu at (136.5, 100.0)
